File: QuadLFO-Dev.brd (EAGLE design)
At the start: 99 x 98.7 mm, 41 parts, among them IC5 MCP6004P, Q2 20MHz, U2 LM4040, U3 328P, U5 7805

Commit message: changed to &4 seris op amps
Parts:
- removed C5: 100n, rcl:C0805K
- removed CV1, CV2, CV3, CV4: PJ302M, GMSN:PJ302M
- removed IC5: MCP6004P, GMSN-R2Project:DIL14
- added C13, C14, C15, C4: 100pF, GMSN:C0805
- added C3: 100nF, GMSN:C0805
- added IC1, IC2, IC3, IC4: TL074, GMSN:SO14
- added OUT, OUT1, OUT2, OUT3: PJ301M-12, GMSN:PJ301M-12
- added R1, R10, R13, R16: 200R, GMSN:R0805
- added R11, R14, R17, R4: 402k, GMSN:R0805
- added R12, R15, R18, R5, R6: 100k, GMSN:R0805
- added R7: 150k, GMSN:R0805
Connections:
- removed net N$13: C2.-, D2.A
- removed net N$25: CV4.TIP, IC5.6, IC5.7
- removed net N$31: CV3.TIP, IC5.1, IC5.2
- removed net N$36: CV2.TIP, IC5.13, IC5.14
- removed net N$7: CV1.TIP, IC5.8, IC5.9
- new net -12V: C2.-, D2.A, IC1.11
- new net N$12: C13.1, IC3.2, R4.1, R6.2
- new net N$14: C4.2, IC1.1, R10.1, R11.2
- new net N$15: OUT1.TIP, R10.2
- new net N$18: C4.1, IC1.2, R11.1, R12.2
- new net N$19: C14.2, IC2.1, R13.1, R14.2
- new net N$20: OUT2.TIP, R13.2
- new net N$23: C14.1, IC2.2, R14.1, R15.2
- new net N$24: C15.2, IC4.1, R16.1, R17.2
- new net N$26: OUT3.TIP, R16.2
- new net N$27: C3.1, IC1.3, IC2.3, IC3.3, IC4.3, R5.2, R7.1
- new net N$29: C15.1, IC4.2, R17.1, R18.2
- new net N$4: C13.2, IC3.1, R1.1, R4.2
- new net N$5: OUT.TIP, R1.2
- new net V+: IC2.4, IC3.4, IC4.4
- new net V-: IC2.11, IC3.11, IC4.11
- net 12V: now also IC1.4
- net 5V: now also R7.2; no longer C5.1, IC5.4
- net GND: now also C3.2, OUT.GND, OUT1.GND, OUT2.GND, OUT3.GND, R5.1; no longer C5.2, CV1.GND, CV2.GND, CV3.GND, CV4.GND, IC5.11
- net VOUTA: now also R6.1; no longer IC5.10
- net VOUTB: now also R12.1; no longer IC5.12
- net VOUTC: now also R15.1; no longer IC5.3
- net VOUTD: now also R18.1; no longer IC5.5
