File: QuadLFO-Dev.sch (EAGLE design)
At the start: 41 parts, among them IC5 MCP6004P, Q2 20MHz, U2 LM4040, U3 328P, U5 7805

Commit message: changed to &4 seris op amps
Parts:
- removed C5: 100n, rcl:C-USC0805K
- removed CV1, CV2, CV3, CV4: PJ302M, GMSN:PJ302M
- removed IC5: MCP6004P, GMSN-R2Project:MCP6004P
- added C13, C14, C15, C4: 100pF, GMSN:CAPACITOR-USC0805
- added C3: 100nF, GMSN:CAPACITOR-USC0805
- added IC1, IC2, IC3, IC4: TL074, GMSN:OPAMP_QUADD
- added OUT, OUT1, OUT2, OUT3: PJ301M-12, GMSN:SOCKET_MONO_3.5MMPJ301M-12
- added R1, R10, R13, R16: 200R, GMSN:RESISTOR_USR0805
- added R11, R14, R17, R4: 402k, GMSN:RESISTOR_USR0805
- added R12, R15, R18, R5, R6: 100k, GMSN:RESISTOR_USR0805
- added R7: 150k, GMSN:RESISTOR_USR0805
Connections:
- removed net N$13: C2.-, D2.A
- removed net N$25: CV4.TIP, IC5B.-IN, IC5B.OUT
- removed net N$31: CV3.TIP, IC5A.-IN, IC5A.OUT
- removed net N$36: CV2.TIP, IC5D.-IN, IC5D.OUT
- removed net N$7: CV1.TIP, IC5C.-IN, IC5C.OUT
- new net -12V: C2.-, D2.A, IC1P.V-
- new net N$12: C13.1, IC3A.-IN, R4.1, R6.2
- new net N$14: C4.2, IC1A.OUT, R10.1, R11.2
- new net N$15: OUT1.TIP, R10.2
- new net N$18: C4.1, IC1A.-IN, R11.1, R12.2
- new net N$19: C14.2, IC2A.OUT, R13.1, R14.2
- new net N$20: OUT2.TIP, R13.2
- new net N$23: C14.1, IC2A.-IN, R14.1, R15.2
- new net N$24: C15.2, IC4A.OUT, R16.1, R17.2
- new net N$26: OUT3.TIP, R16.2
- new net N$27: C3.1, IC1A.+IN, IC2A.+IN, IC3A.+IN, IC4A.+IN, R5.2, R7.1
- new net N$29: C15.1, IC4A.-IN, R17.1, R18.2
- new net N$4: C13.2, IC3A.OUT, R1.1, R4.2
- new net N$5: OUT.TIP, R1.2
- net 12V: now also IC1P.V+
- net 5V: now also R7.2; no longer C5.1, IC5P.V+
- net GND: now also C3.2, OUT.SLEEVE, OUT1.SLEEVE, OUT2.SLEEVE, OUT3.SLEEVE, R5.1; no longer C5.2, CV1.SLEEVE, CV2.SLEEVE, CV3.SLEEVE, CV4.SLEEVE, IC5P.V-
- net VOUTA: now also R6.1; no longer IC5C.+IN
- net VOUTB: now also R12.1; no longer IC5D.+IN
- net VOUTC: now also R15.1; no longer IC5A.+IN
- net VOUTD: now also R18.1; no longer IC5B.+IN
